File: kicad/fpvc-power-distribution.kicad_sch (KiCad schematic)
At the start: 47 parts, among them J1 Solenoid1, J10 PLC_In, J11 PLC_Out, J2 Vout_Screen, J3 Solenoid1, J5 Clutch, J7 Vin_24V, Q1 IRLZ44N, Q2 IRLZ44N, Q4 IRLZ44N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

Commit message: feat: Fix annotations and footprint assignments
Parts:
- C1: renamed from C2; footprint (none) -> Capacitor_SMD:CP_Elec_8x6.2
- C2: renamed from C1; footprint (none) -> Capacitor_SMD:C_0805_2012Metric_Pad1.18x1.45mm_HandSolder
- C3, C4, C6, C8: footprint (none) -> Capacitor_SMD:CP_Elec_8x6.2
- C5, C7, C9: footprint (none) -> Capacitor_SMD:C_0805_2012Metric_Pad1.18x1.45mm_HandSolder
- D4: renamed from D5; footprint (none) -> LED_THT:LED_D5.0mm
- D5: renamed from D6; footprint (none) -> LED_THT:LED_D5.0mm
- D6: renamed from D7; footprint (none) -> LED_THT:LED_D5.0mm
- D7: renamed from D4; footprint (none) -> LED_THT:LED_D5.0mm
- F1: renamed from F4; footprint (none) -> Fuse:Fuseholder_Blade_Mini_Keystone_3568
- F2: renamed from F1; footprint (none) -> Fuse:Fuse_2920_7451Metric_Pad2.10x5.45mm_HandSolder
- F3: renamed from F2; footprint (none) -> Fuse:Fuse_2920_7451Metric_Pad2.10x5.45mm_HandSolder
- F4: renamed from F3; value 8A Polyfuse -> 8A Fuse; footprint (none) -> Fuse:Fuseholder_Blade_Mini_Keystone_3568
- J1, SW1: footprint (none) -> footprints:TE_3-1437652-9
- J2: renamed from J3; footprint (none) -> footprints:TE_3-1437652-9
- J3: renamed from J5; footprint (none) -> footprints:TE_3-1437652-9
- J4: renamed from J10; footprint (none) -> footprints:PHOENIX_1881503
- J5: renamed from J11; footprint (none) -> footprints:PHOENIX_1881503
- J6: renamed from J7; footprint (none) -> footprints:TE_3-1437652-9
- J7: renamed from J2; footprint (none) -> Connector_PinHeader_2.54mm:PinHeader_1x02_P2.54mm_Vertical
- Q1, Q2: value IRLZ44N -> IRLB8314
- Q3: renamed from Q4; value IRLZ44N -> IRLB8314
- R1, R10, R2, R3, R4, R5, R6, R7, R8, R9: footprint (none) -> Resistor_SMD:R_0805_2012Metric_Pad1.20x1.40mm_HandSolder
- R11: renamed from R13; footprint (none) -> Resistor_SMD:R_0805_2012Metric_Pad1.20x1.40mm_HandSolder
- R12: renamed from R11; footprint (none) -> Resistor_SMD:R_0805_2012Metric_Pad1.20x1.40mm_HandSolder
- R13: renamed from R12; footprint (none) -> Resistor_SMD:R_0805_2012Metric_Pad1.20x1.40mm_HandSolder
- SW2: renamed from SW3; footprint (none) -> footprints:TE_3-1437652-9
- U1: footprint (none) -> footprints:D42V110F12
Connections:
- net GND: now also J7.2 (Pin_2); no longer J7.1 (Pin_1)
- net at C8.1, C9.1: now also J7.1 (Pin_1); no longer J7.2 (Pin_2)
Other:
- moved on the sheet: C8, C9, J4, J5, J6, J7, R12, R13, SW1, SW2

Commit message: feat: Finish PCB revision 1
Parts:
- added J10: Load Drivers, footprints:8.26mm Pitch Beau PCB Terminal Strip, symbol Connector:Screw_Terminal_01x06
- added J8: PG, Connector_PinHeader_2.00mm:PinHeader_1x01_P2.00mm_Vertical, symbol Connector:Conn_01x01_Pin
- added J9: GPIO, footprints:8.26mm Pitch Beau PCB Terminal Strip, symbol Connector:Screw_Terminal_01x06
- J2: value Solenoid1 -> Solenoid2
- Q1, Q2, Q3: footprint Package_TO_SOT_THT:TO-220-3_Vertical -> Package_TO_SOT_THT:TO-220-3_Horizontal_TabDown
Connections:
- net GND: now also C1.2, C2.2, J9.5 (Pin_5)
- net PLC_SW1: now also J9.3 (Pin_3)
- net PLC_SW2: now also J9.1 (Pin_1)
- net V_Fault: now also J8.1 (Pin_1)
- net Sol2-1: now reaches D2.1 (K), F3.2, J2.1 (Pin_1)
- net Sol2-1: now also J10.3 (Pin_3)
- net Sol2-2: now reaches D2.2 (A), J2.2 (Pin_2), Q2.2 (D)
- net Sol2-2: now also J10.4 (Pin_4)
- net S1-G: now reaches Q1.1 (G), R1.2, R2.1
- net VIN: now reaches F1.1
- net VIN: now also J6.1 (Pin_1), J9.6 (Pin_6)
- net 24V: now reaches C1.1, C2.1, F1.2
- net 24V: now also C8.1, C9.1, D5.2 (A), F2.1, F3.1, J7.1 (Pin_1), SW1.1 (A), SW2.1 (A), U1.1 (Vin), J9.2 (Pin_2), J9.4 (Pin_4)
- net C-G: now reaches Q3.1 (G), R5.2, R6.1
- net Clu-2: now reaches D3.2 (A), J3.2 (Pin_2), Q3.2 (D)
- net Clu-2: now also J10.6 (Pin_6)
- net Sol1-1: now reaches D1.1 (K), F2.2, J1.1 (Pin_1)
- net Sol1-1: now also J10.1 (Pin_1)
- net Sol1-2: now reaches D1.2 (A), J1.2 (Pin_2), Q1.2 (D)
- net Sol1-2: now also J10.2 (Pin_2)
- net S2-G: now reaches Q2.1 (G), R3.2, R4.1
- net Clu-1: now reaches D3.1 (K), F4.2, J3.1 (Pin_1)
- net Clu-1: now also J10.5 (Pin_5)
Other:
- moved on the sheet: C1, C2, F1, J1, J2, J3, J6
